File: PCB-dual/trackball.kicad_sch (KiCad schematic)
At the start: 7 parts, among them J1 Conn_01x01_Male, J2 Conn_01x01_Male, J3 Conn_01x01_Male, Q1 MMBT2222A-7-F, U1 Adafruit_QT_Py_M0, U2 MrJohnK_PMW3360DM-T2QU, U3 MrJohnK_PMW3360DM-T2QU

Commit message: feat: v1.4 with ~3.4mm spacing between sensor header pins on center with new case optimization, QTPy positioning fix, new ground pad for grounding to case, few track tweaks
Parts:
- added H1: MountingHole_Pad, MountingHole:MountingHole_3.2mm_M3_Pad, symbol Mechanical:MountingHole_Pad
Connections:
- net GND: no longer names the net of Q1.2 (E), U1.9 (GND), U2.2 (GD), U3.2 (GD)
- net GND: now also H1.1
Changed lines of the file:
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@@
+    (stroke (width 0) (type default) (color 0 0 0 0))
+  )
+  (wire (pts (xy 163.83 87.63) (xy 189.23 87.63))
     (stroke (width 0) (type default) (color 0 0 0 0))
   )
@@
   )
   (wire (pts (xy 176.53 109.22) (xy 168.91 109.22))
-    (stroke (width 0) (type default) (color 0 0 0 0))
-  )
-  (wire (pts (xy 170.18 87.63) (xy 163.83 87.63))
     (stroke (width 0) (type default) (color 0 0 0 0))
   )
@@
     (pin "1")
   )
+  (symbol (lib_id "Mechanical:MountingHole_Pad") (at 191.77 87.63 270) (unit 1)
+    (in_bom yes) (on_board yes)
+    (property "Reference" "H1" (id 0) (at 195.58 86.3599 90)
+      (effects (font (size 1.27 1.27)) (justify left))
+    )
+    (property "Value" "MountingHole_Pad" (id 1) (at 195.58 88.8999 90)
+      (effects (font (size 1.27 1.27)) (justify left))
+    )
+    (property "Footprint" "MountingHole:MountingHole_3.2mm_M3_Pad" (id 2) (at 207.01 83.82 90))
+    (property "Datasheet" "~" (id 3) (at 191.77 87.63 0)
+      (effects (font (size 1.27 1.27)) hide)
+    )
+    (pin "1")
+  )
   (symbol (lib_id "Adafruit QT Py M0:MrJohnK_PMW3360DM-T2QU") (at 171.45 138.43 0) (unit 1)
     (in_bom yes) (on_board yes) (fields_autoplaced)
@@
     (pin "1")
   )
-  (symbol (lib_id "power:GND") (at 170.18 87.63 90) (unit 1)
-    (in_bom yes) (on_board yes) (fields_autoplaced)
-    (property "Reference" "#PWR01" (id 0) (at 176.53 87.63 0)
-      (effects (font (size 1.27 1.27)) hide)
-    )
-    (property "Value" "GND" (id 1) (at 173.99 87.6299 90)
-      (effects (font (size 1.27 1.27)) (justify right))
-    )
-    (property "Footprint" "" (id 2) (at 170.18 87.63 0)
-      (effects (font (size 1.27 1.27)) hide)
-    )
-    (property "Datasheet" "" (id 3) (at 170.18 87.63 0)
-      (effects (font (size 1.27 1.27)) hide)
-    )
-    (pin "1")
-  )
   (sheet_instances
     (path "/" (page "1"))
   )
   (symbol_instances
-    (path "/d5da1c1d-0c32-4c68-a42d-2f8e4e93789a"
-      (reference "#PWR01") (unit 1) (value "GND") (footprint "")
+    (path "/950e0eb5-4345-49cd-bfcf-4853d469c843"
+      (reference "H1") (unit 1) (value "MountingHole_Pad") (footprint "MountingHole:MountingHole_3.2mm_M3_Pad")
     )
     (path "/c2d49b82-64df-48fc-9101-7ff2b97b4c1c"
